File: esp32c3-at-adapter.kicad/esp32c3-at-adapter.kicad_sch (KiCad schematic)
At the start: 6 parts, among them J1 Grove, J2 Conn_01x02, U1 ESP32-C3_SUPERMINI

Commit message: Rev: 0.90 (first production test)
Parts:
- removed J1: Grove, user:Grove_1x04_P2mm_Horizontal, symbol user:Grove
- added J1: Stemma-QT_Qwicc, user:JST_SH_SM04B-SRSS-TB_1x04-1MP_P1.00mm_Horizontal, symbol user:Stemma-QT_Qwicc
- H1, H2, U1: now left out of the parts list
- J2: value Conn_01x02 -> WakePins; footprint Connector_JST:JST_XH_S2B-XH-A_1x02_P2.50mm_Horizontal -> Connector_PinHeader_2.54mm:PinHeader_1x02_P2.54mm_Vertical; now left out of the parts list
- JP1: value Jumper_3_Bridged12 -> PWR_Select; now left out of the parts list
Connections:
- net +3V3: now also JP1.1 (A); no longer JP1.2 (C)
- net ESP_RX: now also J1.3 (SDA)
- net ESP_TX: now also J1.4 (SCL)
- net GND: now also J1.1 (GND)
- net VCC: now also JP1.2 (C), J1.2 (Vcc); no longer JP1.1 (A)
Other:
- note added: "As co-processor with AT-firmware it is possible to power the SuperMini via 5V. Change the jumper if the 3V3 is not stable enough."
- note added: "The Stemma/Qt will work as I2C-connector if the SuperMini is used in MCU host mode. Otherwise (as Wifi co-processor with AT-firmware), the connector will link to UART1. On host MCU side, make sure that VCC is connected to the correct power pin and connect SDA of the Stemma/Qt to an UART-TX and SCL to an UART-RX pin."
- moved on the sheet: J2, JP1, U1
